Commit message: Bugs fixed and IMU functionality added.

File: src/robot_description/urdf/3drobot.xacro (robot description, xacro)
@@ -5,10 +5,5 @@
 	xmlns:interface="http://playerstage.sourceforge.net/gazebo/xmlschema/#interface"
 	name="3drobot_xacro">
-	<!--Useful parameters definition.-->
-	<xacro:property name="length_wheel" value="0.03935" />
-	<xacro:property name="radius_wheel" value="0.041275" />
-	<xacro:property name="origin_x_Wheel_collision" value="0"/>
-	<xacro:property name="origin_y_Wheel_collision" value="0"/>
-	<xacro:property name="origin_z_Wheel_collision" value="0"/>
+	<!--Color description.-->
 	<material name="gray">
 	<color rgba="0.58 0.65 0.65 1"/>
@@ -25,5 +20,5 @@
 				<mesh filename="package://robot_description/meshes/base.STL" scale="0.001 0.001 0.001"/>
 			</geometry>
-			<origin rpy="1.5708 0 0" xyz="-0.14364 0.14364 0.0157"/>
+			<origin rpy="0 0 0" xyz="-0.14364 -0.14364 0.0157"/>
 			<material name="gray"/>
 		</visual>
@@ -49,7 +44,7 @@
 		<collision>
 			<geometry>
-				<cylinder length="${length_wheel}" radius="${radius_wheel}"/>
-			</geometry>
-			<origin rpy="1.5708 0 0" xyz="${origin_x_Wheel_collision} ${origin_y_Wheel_collision} ${origin_z_Wheel_collision}"/>
+				<cylinder length="0.03935" radius="0.041275"/>
+			</geometry>
+			<origin rpy="1.5708 0 0" xyz="0 0 0"/>
 		</collision>
 		<inertial>
@@ -68,7 +63,7 @@
 			<collision>
 			<geometry>
-				<cylinder length="${length_wheel}" radius="${radius_wheel}"/>
-			</geometry>
-			<origin rpy="1.5708 0 0" xyz="${origin_x_Wheel_collision} ${origin_y_Wheel_collision} ${origin_z_Wheel_collision}"/>
+				<cylinder length="0.03935" radius="0.041275"/>
+			</geometry>
+			<origin rpy="1.5708 0 0" xyz="0 0 0"/>
 		</collision>
 		<inertial>
@@ -87,7 +82,7 @@
 		<collision>
 			<geometry>
-				<cylinder length="${length_wheel}" radius="${radius_wheel}"/>
-			</geometry>
-			<origin rpy="1.5708 0 0" xyz="${origin_x_Wheel_collision} ${origin_y_Wheel_collision} ${origin_z_Wheel_collision}"/>
+				<cylinder length="0.03935" radius="0.041275"/>
+			</geometry>
+			<origin rpy="1.5708 0 0" xyz="0 0 0"/>
 		</collision>
 		<inertial>
@@ -106,7 +101,7 @@
 		<collision>
 			<geometry>
-				<cylinder length="${length_wheel}" radius="${radius_wheel}"/>
-			</geometry>
-			<origin rpy="1.5708 0 0" xyz="${origin_x_Wheel_collision} ${origin_y_Wheel_collision} ${origin_z_Wheel_collision}"/>
+				<cylinder length="0.03935" radius="0.041275"/>
+			</geometry>
+			<origin rpy="1.5708 0 0" xyz="0 0 0"/>
 		</collision>
 		<inertial>
@@ -118,5 +113,5 @@
 		<visual>
 			<geometry>
-				<mesh filename="package://robot_description/meshes/ejez.STL" scale="0.001 0.001 0.001"/>
+				<mesh filename="package://robot_description/meshes/z_axis.STL" scale="0.001 0.001 0.001"/>
 			</geometry>
 			<origin rpy="0 0 0" xyz="-0.01 -0.05976 0"/>
@@ -153,4 +148,23 @@
 		</inertial>
 	</link>
+	<link name="imu_link">
+   		<visual>
+     		<geometry>
+       			<box size="0.04 0.02 0.001"/>
+     		</geometry>
+			<origin rpy="0 0 0" xyz="0 0 0"/>
+			<material name="gray2"/>>
+		</visual>
+		<collision>
+			<geometry>
+       			<box size="0.04 0.02 0.001"/>
+			</geometry>
+			<origin rpy="0 0 0" xyz="0 0 0"/>
+		</collision>
+		<inertial>
+			<mass value="1e-5" />
+	 		<inertia ixx="1e-6" ixy="0" ixz="0" iyy="1e-6" iyz="0" izz="1e-6" />
+		</inertial>
+ 	</link>
 	<!--Joints definition.-->
 	<joint name="base_to_wheel1" type="continuous">
@@ -189,4 +203,10 @@
 		<origin rpy="0 0 0" xyz="0.075 0 -0.04115"/>
 		<limit effort="1000.0" lower="0.18" upper="0.2" velocity="0.001"/>
+		<axis xyz="0 0 1" />
+	</joint>
+	<joint name="imu_joint" type="fixed">
+		<parent link="base_link"/>
+		<child link="imu_link"/>
+		<origin rpy="0 0 0" xyz="0 0 0.079"/>
 		<axis xyz="0 0 1" />
 	</joint>

Commit message: Packages reorganized and a README added for each one, change of the robot model (TODO: fix the URDF.), firmware implementation in Arduino, improved robot control, installation bash file created and GCode parser.

File: src/robot_description/urdf/3drobot.xacro (robot description, xacro)
@@ -20,16 +20,16 @@
 				<mesh filename="package://robot_description/meshes/base.STL" scale="0.001 0.001 0.001"/>
 			</geometry>
-			<origin rpy="0 0 0" xyz="-0.14364 -0.14364 0.0157"/>
+			<origin rpy="0 0 0" xyz="-0.14364 -0.14364 0"/>
 			<material name="gray"/>
 		</visual>
 		<collision>
 			<geometry>
-				<box size="0.287279 0.287279 0.239"/>
-			</geometry>
-			<origin rpy="0 0 0" xyz="0 0 0.135"/>
-		</collision>
-		<inertial>
-			<mass value="1.78"/>
-			<inertia ixx="0.01336" ixy="0.0" ixz="-0.00008" iyx="0.0" iyy="0.01357" iyz="-0.00002" izx="-0.00008" izy="-0.00002" izz="0.01323"/>
+				<box size="0.287278 0.287278 0.33650"/>
+			</geometry>
+			<origin rpy="0 0 0" xyz="-0.14364 -0.14364 0"/>
+		</collision>
+		<inertial>
+			<mass value="2.55278"/>
+			<inertia ixx="0.01981" ixy="-0.00001" ixz="0.00052" iyx="-0.00001" iyy="0.01998" iyz="0.00040" izx="0.00052" izy="0.00040" izz="0.01846"/>
 		</inertial>
 	</link>
@@ -39,16 +39,16 @@
 				<mesh filename="package://robot_description/meshes/omniwheel.STL" scale="0.001 0.001 0.001"/>
 			</geometry>
-			<origin rpy="1.5708 0 0" xyz="-0.046275 0.019675 -0.046275"/>
-			<material name="gray2"/>>
-		</visual>
-		<collision>
-			<geometry>
-				<cylinder length="0.03935" radius="0.041275"/>
-			</geometry>
-			<origin rpy="1.5708 0 0" xyz="0 0 0"/>
-		</collision>
-		<inertial>
-			<mass value="0.127"/>
-			<inertia ixx="0.00007" ixy="0.0" ixz="0.0" iyy="0.00011" iyz="0.0" izz="0.00007"/>
+			<origin rpy="1.5708 0 0" xyz="0 0 0"/>
+			<material name="gray2"/>>
+		</visual>
+		<collision>
+			<geometry>
+				<cylinder length="0.03935" radius="0.041275"/>
+			</geometry>
+			<origin rpy="1.5708 0 0" xyz="0 0 0"/>
+		</collision>
+		<inertial>
+			<mass value="0.12550"/>
+			<inertia ixx="0.00006" ixy="0.00000" ixz="0.00000" iyx="0.00000" iyy="0.00006" iyz="0.00000" izx="0.00000" izy="0.00000" izz="0.00010"/>
 		</inertial>
 	</link>
@@ -58,5 +58,5 @@
 				<mesh filename="package://robot_description/meshes/omniwheel.STL" scale="0.001 0.001 0.001"/>
 			</geometry>
-			<origin rpy="1.5708 0 0" xyz="-0.046275 0.019675 -0.046275"/>
+			<origin rpy="1.5708 0 0" xyz="0 0 10"/>
 			<material name="gray2"/>>
 		</visual>
@@ -68,6 +68,6 @@
 		</collision>
 		<inertial>
-			<mass value="0.127"/>
-			<inertia ixx="0.00007" ixy="0.0" ixz="0.0" iyy="0.00011" iyz="0.0" izz="0.00007"/>
+			<mass value="0.12550"/>
+			<inertia ixx="0.00006" ixy="0.00000" ixz="0.00000" iyx="0.00000" iyy="0.00006" iyz="0.00000" izx="0.00000" izy="0.00000" izz="0.00010"/>
 		</inertial>
 	</link>
@@ -77,16 +77,16 @@
 				<mesh filename="package://robot_description/meshes/omniwheel.STL" scale="0.001 0.001 0.001"/>
 			</geometry>
-			<origin rpy="1.5708 0 0" xyz="-0.046275 0.019675 -0.046275"/>
-			<material name="gray2"/>>
-		</visual>
-		<collision>
-			<geometry>
-				<cylinder length="0.03935" radius="0.041275"/>
-			</geometry>
-			<origin rpy="1.5708 0 0" xyz="0 0 0"/>
-		</collision>
-		<inertial>
-			<mass value="0.127"/>
-			<inertia ixx="0.00007" ixy="0.0" ixz="0.0" iyy="0.00011" iyz="0.0" izz="0.00007"/>
+			<origin rpy="1.5708 0 0" xyz="0 0 10"/>
+			<material name="gray2"/>>
+		</visual>
+		<collision>
+			<geometry>
+				<cylinder length="0.03935" radius="0.041275"/>
+			</geometry>
+			<origin rpy="1.5708 0 0" xyz="0 0 0"/>
+		</collision>
+		<inertial>
+			<mass value="0.12550"/>
+			<inertia ixx="0.00006" ixy="0.00000" ixz="0.00000" iyx="0.00000" iyy="0.00006" iyz="0.00000" izx="0.00000" izy="0.00000" izz="0.00010"/>
 		</inertial>
 	</link>
@@ -96,16 +96,16 @@
 				<mesh filename="package://robot_description/meshes/omniwheel.STL" scale="0.001 0.001 0.001"/>
 			</geometry>
-			<origin rpy="1.5708 0 0" xyz="-0.046275 0.019675 -0.046275"/>
-			<material name="gray2"/>>
-		</visual>
-		<collision>
-			<geometry>
-				<cylinder length="0.03935" radius="0.041275"/>
-			</geometry>
-			<origin rpy="1.5708 0 0" xyz="0 0 0"/>
-		</collision>
-		<inertial>
-			<mass value="0.127"/>
-			<inertia ixx="0.00007" ixy="0.0" ixz="0.0" iyy="0.00011" iyz="0.0" izz="0.00007"/>
+			<origin rpy="1.5708 0 0" xyz="0 0 10"/>
+			<material name="gray2"/>>
+		</visual>
+		<collision>
+			<geometry>
+				<cylinder length="0.03935" radius="0.041275"/>
+			</geometry>
+			<origin rpy="1.5708 0 0" xyz="0 0 0"/>
+		</collision>
+		<inertial>
+			<mass value="0.12550"/>
+			<inertia ixx="0.00006" ixy="0.00000" ixz="0.00000" iyx="0.00000" iyy="0.00006" iyz="0.00000" izx="0.00000" izy="0.00000" izz="0.00010"/>
 		</inertial>
 	</link>
@@ -115,5 +115,5 @@
 				<mesh filename="package://robot_description/meshes/z_axis.STL" scale="0.001 0.001 0.001"/>
 			</geometry>
-			<origin rpy="0 0 0" xyz="-0.01 -0.05976 0"/>
+			<origin rpy="0 0 0" xyz="0 0 10"/>
 			<material name="gray2"/>>
 		</visual>
@@ -125,6 +125,6 @@
 		</collision>
 		<inertial>
-			<mass value="0.19422"/>
-			<inertia ixx="0.00274" ixy="0.0" ixz="0.00002" iyx="0.0" iyy="0.00259" iyz="0.0" izx="0.00002" izy="0.0" izz="0.00018"/>
+			<mass value="0.17610"/>
+			<inertia ixx="0.00291" ixy="0.00000" ixz="0.00001" iyx="0.00000" iyy="0.00283" iyz="0.00000" izx="0.00001" izy="0.00000" izz="0.00014"/>
 		</inertial>
 	</link>
@@ -134,5 +134,5 @@
 				<mesh filename="package://robot_description/meshes/hotend.STL" scale="0.001 0.001 0.001"/>
 			</geometry>
-			<origin rpy="0 0 0" xyz="-0.068 -0.0599 0.006"/>
+			<origin rpy="0 0 0" xyz="0 0 10"/>
 			<material name="gray2"/>>
 		</visual>
@@ -144,25 +144,25 @@
 		</collision>
 		<inertial>
-			<mass value="0.022"/>
-			<inertia ixx="0.00008" ixy="0.0" ixz="-0.00003" iyx="0.0" iyy="0.00008" iyz="0.0" izx="-0.00003" izy="0.0" izz="0.00010"/>
+			<mass value="0.09737"/>
+			<inertia ixx="0.00009" ixy="0.000000" ixz="-0.00003" iyx="0.00000" iyy="0.00010" iyz="0.00000" izx="-0.00003" izy="0.00000" izz="0.00012"/>
 		</inertial>
 	</link>
 	<link name="imu_link">
-   		<visual>
-     		<geometry>
+		<visual>
+			<geometry>
+				<mesh filename="package://robot_description/meshes/imu.STL" scale="0.001 0.001 0.001"/>
+			</geometry>
+			<origin rpy="0 0 0" xyz="0 0 10"/>
+			<material name="gray2"/>>
+		</visual>
+		<collision>
+			<geometry>
        			<box size="0.04 0.02 0.001"/>
-     		</geometry>
+			</geometry>
 			<origin rpy="0 0 0" xyz="0 0 0"/>
-			<material name="gray2"/>>
-		</visual>
-		<collision>
-			<geometry>
-       			<box size="0.04 0.02 0.001"/>
-			</geometry>
-			<origin rpy="0 0 0" xyz="0 0 0"/>
-		</collision>
-		<inertial>
-			<mass value="1e-5" />
-	 		<inertia ixx="1e-6" ixy="0" ixz="0" iyy="1e-6" iyz="0" izz="1e-6" />
+		</collision>
+		<inertial>
+			<mass value="0.00218" />
+	 		<inertia ixx="0.00000" ixy="0.00000" ixz="0.00000" iyx="0.00000" iyy="0.00000" iyz="0.00000" izx="0.00000" izy="0.00000" izz="0.00000"/>
 		</inertial>
  	</link>

Commit message: URDF fixed, robot colors changed, Z offset in Gazebo launch adjusted, and Arduino Mega port changed.

File: src/robot_description/urdf/3drobot.xacro (robot description, xacro)
@@ -1,43 +1,41 @@
 <?xml version="1.0"?>
 <robot xmlns:xacro="http://www.ros.org/wiki/xacro"
-	xmlns:sensor="http://playerstage.sourceforge.net/gazebo/xmlschema/#sensor"
-	xmlns:controller="http://playerstage.sourceforge.net/gazebo/xmlschema/#controller"
-	xmlns:interface="http://playerstage.sourceforge.net/gazebo/xmlschema/#interface"
-	name="3drobot_xacro">
-	<!--Color description.-->
+ 	xmlns:sensor="http://playerstage.sourceforge.net/gazebo/xmlschema/#sensor"
+    	xmlns:controller="http://playerstage.sourceforge.net/gazebo/xmlschema/#controller"
+    	xmlns:interface="http://playerstage.sourceforge.net/gazebo/xmlschema/#interface"
+	name="3drobot">
+	<xacro:include filename="$(find robot_description)/urdf/3drobot.gazebo" />
 	<material name="gray">
-	<color rgba="0.58 0.65 0.65 1"/>
+		<color rgba="0.58 0.65 0.65 1"/>
 	</material>
 	<material name="gray2">
-	<color rgba="0.58 0.65 0.65 1"/>
+		<color rgba="0.58 0.65 0.65 1"/>
 	</material>
-	<!--Importations-->
-	<xacro:include filename="$(find robot_description)/urdf/3drobot.gazebo" />
-	<!--Links definition.-->
 	<link name="base_link">
-		<visual>
-			<geometry>
-				<mesh filename="package://robot_description/meshes/base.STL" scale="0.001 0.001 0.001"/>
-			</geometry>
-			<origin rpy="0 0 0" xyz="-0.14364 -0.14364 0"/>
+   		<visual>
+			<geometry>
+      			<mesh filename="package://robot_description/meshes/base.STL" scale="0.001 0.001 0.001"/>
+     		</geometry>
+			<origin rpy="0 0 0" xyz="-0.14364 -0.14364 0.0157"/>
 			<material name="gray"/>
-		</visual>
-		<collision>
-			<geometry>
-				<box size="0.287278 0.287278 0.33650"/>
-			</geometry>
-			<origin rpy="0 0 0" xyz="-0.14364 -0.14364 0"/>
-		</collision>
-		<inertial>
-			<mass value="2.55278"/>
-			<inertia ixx="0.01981" ixy="-0.00001" ixz="0.00052" iyx="-0.00001" iyy="0.01998" iyz="0.00040" izx="0.00052" izy="0.00040" izz="0.01846"/>
-		</inertial>
-	</link>
-	<link name="wheel_1">
-		<visual>
-			<geometry>
-				<mesh filename="package://robot_description/meshes/omniwheel.STL" scale="0.001 0.001 0.001"/>
-			</geometry>
-			<origin rpy="1.5708 0 0" xyz="0 0 0"/>
+   		</visual>
+		<collision>
+			<geometry>
+				<box size="0.287279 0.287279 0.239"/>
+			</geometry>
+			<origin rpy="0 0 0" xyz="0 0 0.135"/>
+		</collision>
+			<inertial>
+			<mass value="1.78"/>
+	 		<inertia ixx="0.01336" ixy="0.0" ixz="-0.00008" iyx="0.0" iyy="0.01357" iyz="-0.00002" izx="-0.00008" izy="-0.00002" izz="0.01323"/>
+		</inertial>
+ 	</link>
+ 	<link name="wheel_1">
+   		<visual>
+     		<geometry>
+       			<mesh filename="package://robot_description/meshes/omniwheel.STL" scale="0.001 0.001 0.001"/>
+				<scale>0.001 0.001 0.001</scale>
+     		</geometry>
+			<origin rpy="1.5708 0 0" xyz="-0.046275 0.019675 -0.046275"/>
 			<material name="gray2"/>>
 		</visual>
@@ -49,123 +47,127 @@
 		</collision>
 		<inertial>
-			<mass value="0.12550"/>
-			<inertia ixx="0.00006" ixy="0.00000" ixz="0.00000" iyx="0.00000" iyy="0.00006" iyz="0.00000" izx="0.00000" izy="0.00000" izz="0.00010"/>
-		</inertial>
-	</link>
-	<link name="wheel_2">
-		<visual>
-			<geometry>
-				<mesh filename="package://robot_description/meshes/omniwheel.STL" scale="0.001 0.001 0.001"/>
-			</geometry>
-			<origin rpy="1.5708 0 0" xyz="0 0 10"/>
-			<material name="gray2"/>>
-		</visual>
-			<collision>
-			<geometry>
-				<cylinder length="0.03935" radius="0.041275"/>
-			</geometry>
-			<origin rpy="1.5708 0 0" xyz="0 0 0"/>
-		</collision>
-		<inertial>
-			<mass value="0.12550"/>
-			<inertia ixx="0.00006" ixy="0.00000" ixz="0.00000" iyx="0.00000" iyy="0.00006" iyz="0.00000" izx="0.00000" izy="0.00000" izz="0.00010"/>
-		</inertial>
-	</link>
-	<link name="wheel_3">
-		<visual>
-			<geometry>
-				<mesh filename="package://robot_description/meshes/omniwheel.STL" scale="0.001 0.001 0.001"/>
-			</geometry>
-			<origin rpy="1.5708 0 0" xyz="0 0 10"/>
-			<material name="gray2"/>>
-		</visual>
-		<collision>
-			<geometry>
-				<cylinder length="0.03935" radius="0.041275"/>
-			</geometry>
-			<origin rpy="1.5708 0 0" xyz="0 0 0"/>
-		</collision>
-		<inertial>
-			<mass value="0.12550"/>
-			<inertia ixx="0.00006" ixy="0.00000" ixz="0.00000" iyx="0.00000" iyy="0.00006" iyz="0.00000" izx="0.00000" izy="0.00000" izz="0.00010"/>
-		</inertial>
-	</link>
-	<link name="wheel_4">
-		<visual>
-			<geometry>
-				<mesh filename="package://robot_description/meshes/omniwheel.STL" scale="0.001 0.001 0.001"/>
-			</geometry>
-			<origin rpy="1.5708 0 0" xyz="0 0 10"/>
-			<material name="gray2"/>>
-		</visual>
-		<collision>
-			<geometry>
-				<cylinder length="0.03935" radius="0.041275"/>
-			</geometry>
-			<origin rpy="1.5708 0 0" xyz="0 0 0"/>
-		</collision>
-		<inertial>
-			<mass value="0.12550"/>
-			<inertia ixx="0.00006" ixy="0.00000" ixz="0.00000" iyx="0.00000" iyy="0.00006" iyz="0.00000" izx="0.00000" izy="0.00000" izz="0.00010"/>
-		</inertial>
-	</link>
+			<mass value="0.127"/>
+	 		<inertia ixx="0.00007" ixy="0.0" ixz="0.0" iyy="0.00011" iyz="0.0" izz="0.00007"/>
+		</inertial>
+ 	</link>
+ 	<link name="wheel_2">
+   		<visual>
+     		<geometry>
+       			<mesh filename="package://robot_description/meshes/omniwheel.STL" scale="0.001 0.001 0.001"/>
+				<scale>0.001 0.001 0.001</scale>
+     		</geometry>
+			<origin rpy="1.5708 0 0" xyz="-0.046275 0.019675 -0.046275"/>
+			<material name="gray2"/>>
+		</visual>
+		<collision>
+			<geometry>
+				   <cylinder length="0.03935" radius="0.041275"/>
+			</geometry>
+			<origin rpy="1.5708 0 0" xyz="0 0 0"/>
+		</collision>
+		<inertial>
+			<mass value="0.127"/>
+	 		<inertia ixx="0.00007" ixy="0.0" ixz="0.0" iyy="0.00011" iyz="0.0" izz="0.00007"/>
+		</inertial>
+ 	</link>
+ 	<link name="wheel_3">
+   		<visual>
+     		<geometry>
+       			<mesh filename="package://robot_description/meshes/omniwheel.STL" scale="0.001 0.001 0.001"/>
+				<scale>0.001 0.001 0.001</scale>
+     		</geometry>
+			<origin rpy="1.5708 0 0" xyz="-0.046275 0.019675 -0.046275"/>
+			<material name="gray2"/>>
+		</visual>
+		<collision>
+			<geometry>
+				   <cylinder length="0.03935" radius="0.041275"/>
+			</geometry>
+			<origin rpy="1.5708 0 0" xyz="0 0 0"/>
+		</collision>
+		<inertial>
+			<mass value="0.127"/>
+	 		<inertia ixx="0.00007" ixy="0.0" ixz="0.0" iyy="0.00011" iyz="0.0" izz="0.00007"/>
+		</inertial>
+ 	</link>
+ 	<link name="wheel_4">
+   		<visual>
+     		<geometry>
+       			<mesh filename="package://robot_description/meshes/omniwheel.STL" scale="0.001 0.001 0.001"/>
+				<scale>0.001 0.001 0.001</scale>
+     		</geometry>
+			<origin rpy="1.5708 0 0" xyz="-0.046275 0.019675 -0.046275"/>
+			<material name="gray2"/>>
+		</visual>
+		<collision>
+			<geometry>
+				   <cylinder length="0.03935" radius="0.041275"/>
+			</geometry>
+			<origin rpy="1.5708 0 0" xyz="0 0 0"/>
+		</collision>
+		<inertial>
+			<mass value="0.127"/>
+	 		<inertia ixx="0.00007" ixy="0.0" ixz="0.0" iyy="0.00011" iyz="0.0" izz="0.00007"/>
+		</inertial>
+ 	</link>
 	<link name="z_axis">
-		<visual>
-			<geometry>
-				<mesh filename="package://robot_description/meshes/z_axis.STL" scale="0.001 0.001 0.001"/>
-			</geometry>
-			<origin rpy="0 0 0" xyz="0 0 10"/>
-			<material name="gray2"/>>
-		</visual>
-		<collision>
-			<geometry>
-				<box size="0.0565 0.119526 0.323"/>
+   		<visual>
+     		<geometry>
+       			<mesh filename="package://robot_description/meshes/ejez.STL" scale="0.001 0.001 0.001"/>
+				<scale>0.001 0.001 0.001</scale>
+     		</geometry>
+			<origin rpy="0 0 0" xyz="-0.01 -0.05976 0"/>
+			<material name="gray2"/>>
+		</visual>
+		<collision>
+			<geometry>
+       			<box size="0.0565 0.119526 0.323"/>
 			</geometry>
 			<origin rpy="0 0 0" xyz="0.027 0 0.163"/>
 		</collision>
 		<inertial>
-			<mass value="0.17610"/>
-			<inertia ixx="0.00291" ixy="0.00000" ixz="0.00001" iyx="0.00000" iyy="0.00283" iyz="0.00000" izx="0.00001" izy="0.00000" izz="0.00014"/>
-		</inertial>
-	</link>
+			<mass value="0.19422"/>
+	 		<inertia ixx="0.00274" ixy="0.0" ixz="0.00002" iyx="0.0" iyy="0.00259" iyz="0.0" izx="0.00002" izy="0.0" izz="0.00018"/>
+		</inertial>
+ 	</link>
 	<link name="hotend">
-		<visual>
-			<geometry>
-				<mesh filename="package://robot_description/meshes/hotend.STL" scale="0.001 0.001 0.001"/>
-			</geometry>
-			<origin rpy="0 0 0" xyz="0 0 10"/>
-			<material name="gray2"/>>
-		</visual>
-		<collision>
-			<geometry>
-				<box size="0.085329 0.119724 0.090945"/>
+   		<visual>
+     		<geometry>
+       			<mesh filename="package://robot_description/meshes/hotend.STL" scale="0.001 0.001 0.001"/>
+				<scale>0.001 0.001 0.001</scale>
+     		</geometry>
+			<origin rpy="0 0 0" xyz="-0.068 -0.0599 0.006"/>
+			<material name="gray2"/>>
+		</visual>
+		<collision>
+			<geometry>
+       			<box size="0.085329 0.119724 0.090945"/>
 			</geometry>
 			<origin rpy="0 0 0" xyz="0 0 0.039215"/>
 		</collision>
 		<inertial>
-			<mass value="0.09737"/>
-			<inertia ixx="0.00009" ixy="0.000000" ixz="-0.00003" iyx="0.00000" iyy="0.00010" iyz="0.00000" izx="-0.00003" izy="0.00000" izz="0.00012"/>
-		</inertial>
-	</link>
+			<mass value="0.022"/>
+	 		<inertia ixx="0.00008" ixy="0.0" ixz="-0.00003" iyx="0.0" iyy="0.00008" iyz="0.0" izx="-0.00003" izy="0.0" izz="0.00010"/>
+		</inertial>
+ 	</link>
 	<link name="imu_link">
-		<visual>
-			<geometry>
-				<mesh filename="package://robot_description/meshes/imu.STL" scale="0.001 0.001 0.001"/>
-			</geometry>
-			<origin rpy="0 0 0" xyz="0 0 10"/>
-			<material name="gray2"/>>
-		</visual>
-		<collision>
-			<geometry>
+   		<visual>
+     		<geometry>
        			<box size="0.04 0.02 0.001"/>
-			</geometry>
+     		</geometry>
 			<origin rpy="0 0 0" xyz="0 0 0"/>
-		</collision>
-		<inertial>
-			<mass value="0.00218" />
-	 		<inertia ixx="0.00000" ixy="0.00000" ixz="0.00000" iyx="0.00000" iyy="0.00000" iyz="0.00000" izx="0.00000" izy="0.00000" izz="0.00000"/>
-		</inertial>
- 	</link>
-	<!--Joints definition.-->
+			<material name="gray2"/>>
+		</visual>
+		<collision>
+			<geometry>
+       			<box size="0.04 0.02 0.001"/>
+			</geometry>
+			<origin rpy="0 0 0" xyz="0 0 0"/>
+		</collision>
+		<inertial>
+			<mass value="1e-5" />
+	 		<inertia ixx="1e-6" ixy="0" ixz="0" iyy="1e-6" iyz="0" izz="1e-6" />
+		</inertial>
+ 	</link>
 	<joint name="base_to_wheel1" type="continuous">
 		<parent link="base_link"/>
@@ -210,5 +212,5 @@
 		<origin rpy="0 0 0" xyz="0 0 0.079"/>
 		<axis xyz="0 0 1" />
-	</joint>
+ 	</joint>
 	<!-- Drive controller -->
 	<gazebo>
@@ -219,5 +221,5 @@
 			<odometryRate>50.0</odometryRate>
 			<robotBaseFrame>base_link</robotBaseFrame>
-			<publishTF>false</publishTF>
+			<publishTF>true</publishTF>
 		</plugin>
 	</gazebo>
